File: cad/Logic Board surface mount/Logic Board.brd (EAGLE design)
At the start: 43 x 46 mm, 23 parts, among them Q1 8/16/20MHz, U1 ATMEGA328, U2 MIC5205

Commit message: Updated board
Parts:
- removed JP5, JP8: FIDUCIALUFIDUCIAL, SparkFun:MICRO-FIDUCIAL
- added C4: 10uF, rcl:C1206
- added J1: (no value), SparkFun-Connectors:SCREWTERMINAL-3.5MM-2
- added M1: WIRELESS-NRF24L01-PA-EXT, diy-modules:WIRELESS-NRD24L01-PA-EXT
- moved JP1 10.2 mm to (25.4, 1.27)
- moved SJ1 2.84 mm to (38.5, 23.5)
- moved C2 2.84 mm to (30.4, 16.5)
- moved C1 2.84 mm to (38.6, 43.7)
- moved C13 2.84 mm to (38.5, 19.7)
- moved LED1 2.84 mm to (34.3, 23.9)
- moved Q1 2.84 mm to (38.9, 26.7)
- moved R1 2.84 mm to (30.2, 22.6)
- moved R2 2.84 mm to (38.6, 40.5)
- moved U2 2.84 mm to (34.3, 21.5)
- moved C19 2.84 mm to (30.0, 21.6)
- moved D3 2.84 mm to (29.5, 44.0)
- moved R3 2.84 mm to (28.9, 22.6)
- moved R6 2.84 mm to (29.5, 40.8)
- moved C10 2.84 mm to (36.0, 25.3)
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- renumbered B1 to B2
Connections:
- new net BOUT: B2.B+, B2.B+@2
- new net GOUT: B2.G+, B2.G+@1
- new net N$10: B2.B-, B2.B-@1
- new net N$5: B2.R-, B2.R-@1
- new net N$9: B2.G-, B2.G-@1
- new net ROUT: B2.R+, B2.R+@1
- net D10: now also M1.4
- net D2: now also M1.8
- net D9: now also M1.3
- net GND: now also C4.2, J1.1, M1.1
- net MISO: now also M1.7
- net MOSI: now also M1.6
- net RAW: now also J1.2
- net SCK: now also M1.5
- net VCC: now also C4.1, M1.2
Routing:
- net D10: track 24.4 -> 0.00 mm, vias 1 -> 0
- net GND: track 9.36 -> 27.1 mm
- net VCC: track 56.8 -> 70.5 mm
- net DTR: track 4.42 -> 17.8 mm
- net D9: track 11.7 -> 0.00 mm
- net A5: track 11.0 -> 0.00 mm, vias 1 -> 0
- net D8: track 9.34 -> 0.00 mm
- net RXI: track 40.2 -> 48.3 mm
- net D7: track 6.99 -> 0.00 mm
- net A4: track 6.04 -> 0.00 mm
- net TXO: track 24.1 -> 29.1 mm
- net D6: track 4.79 -> 0.00 mm
- net A3: track 4.48 -> 0.00 mm
- net SCK: track 9.42 -> 5.20 mm
- net A6: track 3.55 -> 0.00 mm
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Other:
- board text removed: "v14"

Commit message: More board layout changes
Parts:
- moved C4 21.3 mm to (33.0, 11.4), turned to 180 degrees
- moved M1 20.3 mm to (35.6, 33.0)
- moved D3 14.2 mm to (16.8, 37.6), turned to 90 degrees
- moved C1 12.7 mm to (25.9, 43.7)
- moved R2 12.7 mm to (25.9, 40.5)
- moved S1 12.7 mm to (21.5, 43.1)
- moved R6 9.44 mm to (20.6, 37.6), turned to 180 degrees
- moved J1 8.89 mm to (12.7, 43.2)
- moved C13 3.81 mm to (38.5, 23.5)
- moved Q1 3.81 mm to (38.9, 30.5)
- moved R1 3.81 mm to (30.2, 26.4)
- moved R3 3.81 mm to (28.9, 26.4)
- moved U1 3.81 mm to (34.3, 35.6)
- moved C10 3.81 mm to (36.0, 29.1)
- moved C19 3.81 mm to (30.0, 25.4)
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Routing:
- net GND: track 27.1 -> 63.2 mm
- net RESET: track 57.0 -> 66.5 mm
- net RXI: track 48.3 -> 56.1 mm
- net SCK: track 5.20 -> 12.8 mm
- net MISO: track 17.1 -> 11.0 mm
- net VCC: track 70.5 -> 75.0 mm
- net TXO: track 29.1 -> 32.9 mm
- net DTR: track 17.8 -> 21.6 mm
- net MOSI: track 11.7 -> 10.1 mm
- net AREF: track 22.8 -> 23.6 mm
- net N$7: track 1.45 -> 2.08 mm
- added copper zone on layer 1, net VCC
- removed copper zone on layer 1, net GND
Other:
- board text added: "TODO: - Replace all headers with SMT - Replace 0603 components with 1206"

Commit message: More tweaks
Parts:
- removed R1, R3: (no value), SparkFun:0603-RES
- moved D3 2.54 mm to (19.3, 37.6)
- moved R6 2.54 mm to (23.1, 37.6)
Connections:
- removed net A4: R1.1, U1.27
- removed net A5: R3.1, U1.28
- net VCC: no longer R1.2, R3.2
Routing:
- net RAW: track 11.3 -> 46.3 mm, vias 2 -> 3
- net RESET: track 66.5 -> 52.6 mm
- net VCC: track 75.0 -> 70.2 mm
- net GND: track 63.2 -> 65.7 mm
- net SCK: track 12.8 -> 11.2 mm
Changed lines of the file:
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@@
 <attribute name="VALUE" x="24.9428" y="44.4373" size="0.4064" layer="27" rot="R270"/>
 </element>
-<element name="R6" library="SparkFun" package="0603-RES" value="330" x="20.574" y="37.6428" smashed="yes" rot="R180">
-<attribute name="NAME" x="22.574" y="37.6428" size="1.27" layer="25"/>
-<attribute name="VALUE" x="20.2316" y="38.2778" size="0.4064" layer="27"/>
-</element>
-<element name="D3" library="Testing" package="0603-LED-ALT1" value="Green" x="16.764" y="37.6428" smashed="yes" rot="R90">
-<attribute name="NAME" x="18.764" y="37.6428" size="1.27" layer="25"/>
-<attribute name="VALUE" x="16.0152" y="38.3032" size="0.4064" layer="27"/>
+<element name="R6" library="SparkFun" package="0603-RES" value="330" x="23.114" y="37.6428" smashed="yes" rot="R180">
+<attribute name="NAME" x="25.114" y="37.6428" size="1.27" layer="25"/>
+<attribute name="VALUE" x="22.7716" y="38.2778" size="0.4064" layer="27"/>
+</element>
+<element name="D3" library="Testing" package="0603-LED-ALT1" value="Green" x="19.304" y="37.6428" smashed="yes" rot="R90">
+<attribute name="NAME" x="21.304" y="37.6428" size="1.27" layer="25"/>
+<attribute name="VALUE" x="18.5552" y="38.3032" size="0.4064" layer="27"/>
 </element>
 <element name="U2" library="SparkFun" package="SOT23-5" value="MIC5205" x="34.29" y="25.3492" smashed="yes" rot="R270">
@@
 <element name="JP1" library="SparkFun" package="1X06" value="FTDI Basic" x="25.4" y="1.27" rot="MR180"/>
 <element name="C2" library="SparkFun" package="0603-CAP" value="0.1uF" x="30.3784" y="20.32"/>
-<element name="R1" library="SparkFun" package="0603-RES" value="" x="30.2006" y="26.3652" rot="MR270"/>
-<element name="R3" library="SparkFun" package="0603-RES" value="" x="28.9306" y="26.3652" rot="MR270"/>
 <element name="FRAME1" library="SparkFun-Aesthetics" package="CREATIVE_COMMONS" value="FRAME-LETTER" x="-15.982121875" y="-8.89"/>
 <element name="SJ1" library="SparkFun-Passives" package="SJ_2S" value="" x="38.481" y="27.305" rot="R90"/>
@@
 <wire x1="33.313" y1="42.291" x2="31.115" y2="42.291" width="0.254" layer="1"/>
 <wire x1="12.7" y1="43.18" x2="12.7" y2="40.8298" width="0.254" layer="1"/>
-<wire x1="12.7" y1="40.8298" x2="15.887" y2="37.6428" width="0.254" layer="1"/>
 <wire x1="18.669" y1="44.8698" x2="14.3898" y2="44.8698" width="0.254" layer="1"/>
 <wire x1="14.3898" y1="44.8698" x2="12.7" y2="43.18" width="0.254" layer="1"/>
@@
 <wire x1="29.972" y1="26.8" x2="31.7754" y2="25.4" width="0" layer="19" extent="1-1"/>
 <wire x1="33.44" y1="22.86" x2="32.9899" y2="25.3492" width="0" layer="19" extent="1-1"/>
+<wire x1="12.7" y1="40.8298" x2="15.887" y2="37.6428" width="0.254" layer="1"/>
+<wire x1="15.887" y1="37.6428" x2="18.427" y2="37.6428" width="0.254" layer="1"/>
 </signal>
 <signal name="AREF">
@@
 <contactref element="U1" pad="29"/>
 <contactref element="C2" pad="1"/>
-<wire x1="35.433" y1="29.21" x2="38.1" y2="29.21" width="0.254" layer="16"/>
 <wire x1="30.861" y1="31.5653125" x2="30.861" y2="28.448" width="0.254" layer="1"/>
 <wire x1="27.94" y1="27.051" x2="27.94" y2="24.8412" width="0.254" layer="1"/>
@@
 <wire x1="27.4066" y1="23.9522" x2="28.0162" y2="23.3426" width="0.254" layer="1"/>
 <wire x1="28.0162" y1="23.3426" x2="28.0162" y2="21.1074" width="0.254" layer="1"/>
-<wire x1="33.5788" y1="27.3558" x2="35.433" y2="29.21" width="0.254" layer="16"/>
-<wire x1="32.2326" y1="27.3558" x2="33.5788" y2="27.3558" width="0.254" layer="16"/>
-<wire x1="31.8008" y1="27.7876" x2="32.2326" y2="27.3558" width="0.254" layer="16"/>
-<wire x1="31.8008" y1="34.4678" x2="31.8008" y2="27.7876" width="0.254" layer="16"/>
 <wire x1="31.877" y1="34.544" x2="31.8008" y2="34.4678" width="0.254" layer="16"/>
 <via x="27.94" y="41.91" extent="1-16" drill="0.508"/>
@@
 <contactref element="U1" pad="17"/>
 <contactref element="M1" pad="5"/>
-<wire x1="21.424" y1="37.6428" x2="32.356996875" y2="41.4528" width="0.254" layer="1"/>
 <wire x1="32.356996875" y1="41.4528" x2="33.234571875" y2="40.575225" width="0.254" layer="1"/>
-<wire x1="36.83" y1="14.605" x2="33.234571875" y2="40.575225" width="0" layer="19" extent="1-1"/>
+<wire x1="23.964" y1="37.6428" x2="26.2128" y2="37.6428" width="0.254" layer="1"/>
+<wire x1="26.2128" y1="37.6428" x2="30.0228" y2="41.4528" width="0.254" layer="1"/>
+<wire x1="30.0228" y1="41.4528" x2="32.356996875" y2="41.4528" width="0.254" layer="1"/>
+<wire x1="36.83" y1="14.605" x2="26.2128" y2="37.6428" width="0" layer="19" extent="1-1"/>
 </signal>
 <signal name="MISO">
@@
 <contactref element="R6" pad="2"/>
 <contactref element="D3" pad="A"/>
-<wire x1="17.641" y1="37.6428" x2="19.724" y2="37.6428" width="0.254" layer="1"/>
+<wire x1="20.181" y1="37.6428" x2="22.264" y2="37.6428" width="0.254" layer="1"/>
 </signal>
 <signal name="TXO">
@@
 <contactref element="U1" pad="6"/>
 <contactref element="JP1" pad="4"/>
-<contactref element="R3" pad="2"/>
-<contactref element="R1" pad="2"/>
 <wire x1="34.2438" y1="38.4347" x2="34.29" y2="38.3885" width="0.254" layer="1"/>
 <wire x1="34.29" y1="38.4809" x2="34.2438" y2="38.4347" width="0.254" layer="1"/>
@@
 <wire x1="35.052" y1="35.56" x2="35.941" y2="35.56" width="0.254" layer="1"/>
 <wire x1="37.719" y1="35.814" x2="37.719" y2="33.828059375" width="0.254" layer="1"/>
-<wire x1="28.194" y1="25.7302" x2="26.67" y2="27.2542" width="0.254" layer="16"/>
 <wire x1="35.5092" y1="26.289" x2="30.9744" y2="26.289" width="0.254" layer="16"/>
-<wire x1="30.2006" y1="25.5152" x2="28.9306" y2="25.5152" width="0.254" layer="16"/>
 <via x="36.5506" y="27.3304" extent="1-16" drill="0.508"/>
 <wire x1="34.29" y1="38.4809" x2="34.29" y2="41.568" width="0.254" layer="1"/>
@@
 <wire x1="37.04248125" y1="32.241828125" x2="35.941" y2="33.343315625" width="0.254" layer="1"/>
 <wire x1="32.668884375" y1="40.0095375" x2="34.29" y2="38.388428125" width="0.254" layer="1"/>
-<wire x1="30.9744" y1="26.289" x2="30.2006" y2="25.5152" width="0.254" layer="16"/>
-<wire x1="28.194" y1="25.7302" x2="28.7156" y2="25.7302" width="0.254" layer="16"/>
-<wire x1="28.7156" y1="25.7302" x2="28.9306" y2="25.5152" width="0.254" layer="16"/>
 <contactref element="SJ1" pad="2"/>
 <contactref element="C13" pad="A"/>
@@
 <contactref element="C4" pad="1"/>
 <wire x1="34.29" y1="2.54" x2="33.02" y2="1.27" width="0.254" layer="16"/>
-<wire x1="25.9334" y1="39.6376" x2="33.8564" y2="43.4476" width="0.254" layer="1"/>
-<wire x1="33.8564" y1="43.4476" x2="35.013" y2="42.291" width="0.254" layer="1"/>
 <polygon width="0.254" layer="1" isolate="0.3048">
 <vertex x="41.91" y="12.7"/>
@@
 <wire x1="34.42" y1="12.57" x2="33.02" y2="13.97" width="0.254" layer="1"/>
 <wire x1="33.02" y1="13.97" x2="33.02" y2="16.51" width="0.254" layer="1"/>
+<wire x1="35.013" y1="42.291" x2="34.29" y2="43.014" width="0.254" layer="1"/>
+<wire x1="26.67" y1="39.37" x2="26.201" y2="39.37" width="0.254" layer="1"/>
+<wire x1="26.201" y1="39.37" x2="25.9334" y2="39.6376" width="0.254" layer="1"/>
+<wire x1="34.29" y1="43.014" x2="30.314" y2="43.014" width="0.254" layer="1"/>
+<wire x1="30.314" y1="43.014" x2="26.67" y2="39.37" width="0.254" layer="1"/>
 </signal>
 <signal name="RAW" class="1">
@@
 <wire x1="32.9747" y1="24.384" x2="32.9899" y2="24.3992" width="0.254" layer="1"/>
 <contactref element="J1" pad="2"/>
-<wire x1="29.1338" y1="23.1618" x2="9.2" y2="43.18" width="0" layer="19" extent="1-1"/>
+<wire x1="9.2" y1="43.18" x2="9.2" y2="42.87" width="0.254" layer="1"/>
+<wire x1="9.2" y1="42.87" x2="16.51" y2="35.56" width="0.254" layer="1"/>
+<wire x1="16.51" y1="35.56" x2="25.4" y2="35.56" width="0.254" layer="1"/>
+<wire x1="25.4" y1="35.56" x2="26.67" y2="34.29" width="0.254" layer="1"/>
+<wire x1="26.67" y1="34.29" x2="26.67" y2="22.86" width="0.254" layer="1"/>
+<via x="26.67" y="22.86" extent="1-16" drill="0.5"/>
+<wire x1="26.67" y1="22.86" x2="27.9908" y2="22.86" width="0.254" layer="16"/>
+<wire x1="27.9908" y1="22.86" x2="28.6004" y2="22.2504" width="0.254" layer="16"/>
 </signal>
 <signal name="D9">
@@
 <contactref element="U1" pad="12"/>
 </signal>
-<signal name="A5">
-<contactref element="U1" pad="28"/>
-<contactref element="R3" pad="1"/>
-<wire x1="28.9306" y1="27.2152" x2="30.971828125" y2="32.807515625" width="0" layer="19" extent="1-16"/>
-</signal>
-<signal name="A4">
-<contactref element="U1" pad="27"/>
-<contactref element="R1" pad="1"/>
-<wire x1="30.2006" y1="27.2152" x2="30.40614375" y2="33.3732" width="0" layer="19" extent="1-16"/>
-</signal>
 <signal name="A3">
