File: cad/Logic Board surface mount/Logic Board.sch (EAGLE design)
At the start: 23 parts, among them Q1 8/16/20MHz, U1 ATMEGA328, U2 MIC5205

Commit message: Updated board
Parts:
- removed B1: LED-BOARDV4, special:LED-BOARDV4
- removed JP5, JP8: FIDUCIALUFIDUCIAL, SparkFun:FIDUCIALUFIDUCIAL
- added B2: LED-BOARDV4, special:LED-BOARDV4
- added C4: 10uF, rcl:C-USC1206
- added J1: (no value), SparkFun-Connectors:M023.5MM
- added M1: WIRELESS-NRF24L01-PA-EXT, diy-modules:WIRELESS-NRF24L01-PA-EXT
Connections:
- new net BOUT: B2BLUE.P$2
- new net GOUT: B2GREEN.P$2
- new net N$10: B2BLUE.P$1
- new net N$5: B2RED.P$1
- new net N$9: B2GREEN.P$1
- new net ROUT: B2RED.P$2
- net D10: now also M1.CSN
- net D2: now also M1.IRQ
- net D9: now also M1.CE
- net GND: now also C4.2, J1.1, M1.GND
- net MISO: now also M1.MISO
- net MOSI: now also M1.MOSI
- net RAW: now also J1.2
- net SCK: now also M1.SCK
- net VCC: now also C4.1, M1.VCC
Other:
- note removed: "Board outline & LED pads"
- moved on the sheet: JP1

Commit message: More tweaks
Parts:
- removed R1, R3: (no value), SparkFun:RESISTOR0603-RES
Connections:
- removed net A4: R1.1, U1.PC4(ADC4/SDA)
- removed net A5: R3.1, U1.PC5(ADC5/SCL)
- net VCC: no longer R1.2, R3.2
Other:
- note removed: "Optional Pullups for I2C lines"
Changed lines of the file:
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@@
 <part name="JP1" library="SparkFun" deviceset="ARDUINO_SERIAL_PROGRAM" device="PTH" value="FTDI Basic"/>
 <part name="C2" library="SparkFun" deviceset="CAP" device="0603-CAP" value="0.1uF"/>
-<part name="R1" library="SparkFun" deviceset="RESISTOR" device="0603-RES"/>
-<part name="R3" library="SparkFun" deviceset="RESISTOR" device="0603-RES"/>
-<part name="P+2" library="SparkFun" deviceset="3.3V" device="" value="VCC"/>
-<part name="P+3" library="SparkFun" deviceset="3.3V" device="" value="VCC"/>
 <part name="SJ1" library="SparkFun-Passives" deviceset="SOLDERJUMPER" device="NC" value=""/>
 <part name="P+4" library="SparkFun" deviceset="3.3V" device="" value="VCC"/>
@@
 <sheet>
 <plain>
-<wire x1="210.82" y1="177.8" x2="245.872" y2="177.8" width="0.2032" layer="97" style="shortdash"/>
-<wire x1="245.872" y1="177.8" x2="245.872" y2="137.668" width="0.2032" layer="97" style="shortdash"/>
-<wire x1="245.872" y1="137.668" x2="210.82" y2="137.668" width="0.2032" layer="97" style="shortdash"/>
-<wire x1="210.82" y1="137.668" x2="210.82" y2="177.8" width="0.2032" layer="97" style="shortdash"/>
 <text x="165.862" y="11.684" size="1.778" layer="94">Original Arduino Mini Design by Team Arduino</text>
 <text x="165.862" y="9.144" size="1.778" layer="94">Arduino Pro Mini Design by Spark Fun Electronics</text>
@@
 <text x="20.32" y="134.62" size="1.778" layer="97">Max Current Output: 150mA</text>
 <text x="20.32" y="139.7" size="1.778" layer="97">VCC = 5V or 3.3V Output</text>
-<text x="212.598" y="172.72" size="1.778" layer="97">Optional Pullups for I2C lines</text>
 <text x="240.284" y="7.366" size="1.778" layer="94">14</text>
 <text x="58.42" y="177.8" size="1.778" layer="97">Power isolation jumper</text>
@@
 <attribute name="VALUE" x="116.459" y="155.956" size="1.778" layer="96" rot="R90"/>
 </instance>
-<instance part="R1" gate="G$1" x="223.52" y="152.4" rot="R90"/>
-<instance part="R3" gate="G$1" x="231.14" y="149.86" rot="R90"/>
-<instance part="P+2" gate="G$1" x="223.52" y="160.02"/>
-<instance part="P+3" gate="G$1" x="231.14" y="160.02"/>
 <instance part="SJ1" gate="1" x="68.58" y="162.56"/>
 <instance part="P+4" gate="G$1" x="86.36" y="165.1"/>
@@
 <pinref part="JP1" gate="G$1" pin="VCC"/>
 <label x="233.68" y="119.38" size="1.27" layer="95" xref="yes"/>
-</segment>
-<segment>
-<wire x1="223.52" y1="157.48" x2="223.52" y2="160.02" width="0.1524" layer="91"/>
-<pinref part="P+2" gate="G$1" pin="3.3V"/>
-<pinref part="R1" gate="G$1" pin="2"/>
-</segment>
-<segment>
-<wire x1="231.14" y1="154.94" x2="231.14" y2="160.02" width="0.1524" layer="91"/>
-<pinref part="P+3" gate="G$1" pin="3.3V"/>
-<pinref part="R3" gate="G$1" pin="2"/>
 </segment>
 <segment>
@@
 </segment>
 </net>
-<net name="A5" class="0">
-<segment>
-<wire x1="195.58" y1="142.24" x2="231.14" y2="142.24" width="0.1524" layer="91"/>
-<wire x1="231.14" y1="142.24" x2="231.14" y2="144.78" width="0.1524" layer="91"/>
-<pinref part="U1" gate="G$1" pin="PC5(ADC5/SCL)"/>
-<pinref part="R3" gate="G$1" pin="1"/>
-</segment>
-</net>
-<net name="A4" class="0">
-<segment>
-<wire x1="195.58" y1="144.78" x2="223.52" y2="144.78" width="0.1524" layer="91"/>
-<wire x1="223.52" y1="144.78" x2="223.52" y2="147.32" width="0.1524" layer="91"/>
-<pinref part="U1" gate="G$1" pin="PC4(ADC4/SDA)"/>
-<pinref part="R1" gate="G$1" pin="1"/>
-</segment>
-</net>
