File: cad/Base Station/Base Station.sch (EAGLE design)
At the start: 4 parts, among them M1 WIRELESS-NRF24L01-PA-EXT

Commit message: Updated base station
Parts:
- removed JP1: RASPBERRYPI-GPIOPTH, SparkFun-Boards:RASPBERRYPI-GPIOPTH
- removed M1: WIRELESS-NRF24L01-PA-EXT, diy-modules:WIRELESS-NRF24L01-PA-EXT
- added J1: GPIO, pinhead:PINHD-2X13
- added J2: nRF24L01+, my-custom:FEMALE-2X4-SMT
- added LOGO1: OSHW-LOGOS, SparkFun-Aesthetics:OSHW-LOGOS
- C1: device SparkFun-Capacitors:CAP_POLPTH2 -> rcl:C-USC1206K
- FRAME1: value FRAME-LETTER -> FRAME-LETTERNO_PACKAGE; device SparkFun-Aesthetics:FRAME-LETTER -> SparkFun-Aesthetics:FRAME-LETTERNO_PACKAGE
Connections:
- net CE: now also J1.15, J2.3; no longer JP1.GP22, M1.CE
- net CSN: now also J1.24, J2.4; no longer JP1.CE0, M1.CSN
- net GND: now also C1.2, J1.14, J1.20, J1.25, J1.6, J1.9, J2.1; no longer C1.-, JP1.GND@25, M1.GND
- net MISO: now also J1.21, J2.7; no longer JP1.MISO, M1.MISO
- net MOSI: now also J1.19, J2.6; no longer JP1.MOSI, M1.MOSI
- net SCK: now also J1.23, J2.5; no longer JP1.SCLK, M1.SCK
- net VCC: now also C1.1, J1.17, J2.2; no longer C1.+, JP1.3.3V@17, M1.VCC
Changed lines of the file:
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@@
 </classes>
 <parts>
-<part name="FRAME1" library="SparkFun-Aesthetics" deviceset="FRAME-LETTER" device=""/>
-<part name="JP1" library="SparkFun-Boards" deviceset="RASPBERRYPI-GPIO" device="PTH"/>
-<part name="M1" library="diy-modules" deviceset="WIRELESS-NRF24L01-PA-EXT" device=""/>
-<part name="C1" library="SparkFun-Capacitors" deviceset="CAP_POL" device="PTH2" value="10uF"/>
+<part name="FRAME1" library="SparkFun-Aesthetics" deviceset="FRAME-LETTER" device="NO_PACKAGE" value="FRAME-LETTERNO_PACKAGE"/>
+<part name="C1" library="rcl" deviceset="C-US" device="C1206K" value="10uF"/>
+<part name="J2" library="my-custom" deviceset="FEMALE-2X4-SMT" device="" value="nRF24L01+"/>
+<part name="LOGO1" library="SparkFun-Aesthetics" deviceset="OSHW-LOGO" device="S" value="OSHW-LOGOS"/>
+<part name="J1" library="pinhead" deviceset="PINHD-2X13" device="" value="GPIO"/>
 </parts>
 <sheets>
@@
 <instance part="FRAME1" gate="G$1" x="0" y="0"/>
 <instance part="FRAME1" gate="V" x="147.32" y="0"/>
-<instance part="JP1" gate="JP1" x="48.26" y="134.62"/>
-<instance part="M1" gate="G$1" x="182.88" y="124.46"/>
-<instance part="C1" gate="G$1" x="129.54" y="134.62" rot="R180"/>
+<instance part="C1" gate="G$1" x="177.8" y="142.24" smashed="yes" rot="R270">
+<attribute name="NAME" x="175.387" y="137.414" size="1.778" layer="95"/>
+<attribute name="VALUE" x="174.625" y="145.288" size="1.778" layer="96"/>
+</instance>
+<instance part="J2" gate="G$1" x="177.8" y="129.54" rot="R270"/>
+<instance part="LOGO1" gate="G$1" x="231.14" y="48.26"/>
+<instance part="J1" gate="A" x="81.28" y="127" smashed="yes" rot="R90">
+<attribute name="NAME" x="64.008" y="136.779" size="1.778" layer="95"/>
+<attribute name="VALUE" x="63.5" y="119.888" size="1.778" layer="96" rot="MR180"/>
+</instance>
 </instances>
 <busses>
@@
 <net name="VCC" class="0">
 <segment>
-<pinref part="JP1" gate="JP1" pin="3.3V@17"/>
-<wire x1="33.02" y1="152.4" x2="22.86" y2="152.4" width="0.1524" layer="91"/>
-<label x="22.86" y="152.4" size="1.778" layer="95" font="vector"/>
+<pinref part="J2" gate="G$1" pin="2"/>
+<wire x1="185.42" y1="132.08" x2="195.58" y2="132.08" width="0.1524" layer="91"/>
+<label x="195.58" y="132.08" size="1.778" layer="95" font="vector" rot="MR0"/>
+<pinref part="C1" gate="G$1" pin="1"/>
+<wire x1="180.34" y1="142.24" x2="195.58" y2="142.24" width="0.1524" layer="91"/>
+<wire x1="195.58" y1="142.24" x2="195.58" y2="132.08" width="0.1524" layer="91"/>
 </segment>
 <segment>
-<pinref part="M1" gate="G$1" pin="VCC"/>
-<label x="149.86" y="132.08" size="1.778" layer="95" font="vector"/>
-<pinref part="C1" gate="G$1" pin="+"/>
-<wire x1="129.54" y1="132.08" x2="160.02" y2="132.08" width="0.1524" layer="91"/>
+<pinref part="J1" gate="A" pin="17"/>
+<wire x1="86.36" y1="124.46" x2="86.36" y2="111.76" width="0.1524" layer="91"/>
+<label x="86.36" y="111.76" size="1.778" layer="95" font="vector" rot="R90"/>
 </segment>
 </net>
 <net name="GND" class="0">
 <segment>
-<pinref part="JP1" gate="JP1" pin="GND@25"/>
-<wire x1="33.02" y1="111.76" x2="22.86" y2="111.76" width="0.1524" layer="91"/>
-<label x="22.86" y="111.76" size="1.778" layer="95" font="vector"/>
+<wire x1="170.18" y1="132.08" x2="160.02" y2="132.08" width="0.1524" layer="91"/>
+<label x="160.02" y="132.08" size="1.778" layer="95" font="vector"/>
+<pinref part="C1" gate="G$1" pin="2"/>
+<wire x1="160.02" y1="132.08" x2="160.02" y2="142.24" width="0.1524" layer="91"/>
+<wire x1="160.02" y1="142.24" x2="172.72" y2="142.24" width="0.1524" layer="91"/>
+<pinref part="J2" gate="G$1" pin="1"/>
 </segment>
 <segment>
-<pinref part="M1" gate="G$1" pin="GND"/>
-<wire x1="160.02" y1="134.62" x2="142.24" y2="134.62" width="0.1524" layer="91"/>
-<label x="149.86" y="134.62" size="1.778" layer="95" font="vector"/>
-<pinref part="C1" gate="G$1" pin="-"/>
-<wire x1="142.24" y1="134.62" x2="142.24" y2="139.7" width="0.1524" layer="91"/>
-<wire x1="142.24" y1="139.7" x2="129.54" y2="139.7" width="0.1524" layer="91"/>
+<pinref part="J1" gate="A" pin="25"/>
+<wire x1="96.52" y1="124.46" x2="96.52" y2="111.76" width="0.1524" layer="91"/>
+<label x="96.52" y="111.76" size="1.778" layer="95" font="vector" rot="R90"/>
+</segment>
+<segment>
+<pinref part="J1" gate="A" pin="9"/>
+<wire x1="76.2" y1="124.46" x2="76.2" y2="111.76" width="0.1524" layer="91"/>
+<label x="76.2" y="111.76" size="1.778" layer="95" font="vector" rot="R90"/>
+</segment>
+<segment>
+<pinref part="J1" gate="A" pin="6"/>
+<wire x1="71.12" y1="132.08" x2="71.12" y2="144.78" width="0.1524" layer="91"/>
+<label x="71.12" y="144.78" size="1.778" layer="95" font="vector" rot="MR270"/>
+</segment>
+<segment>
+<pinref part="J1" gate="A" pin="14"/>
+<wire x1="81.28" y1="132.08" x2="81.28" y2="144.78" width="0.1524" layer="91"/>
+<label x="81.28" y="144.78" size="1.778" layer="95" font="vector" rot="MR270"/>
+</segment>
+<segment>
+<pinref part="J1" gate="A" pin="20"/>
+<wire x1="88.9" y1="132.08" x2="88.9" y2="144.78" width="0.1524" layer="91"/>
+<label x="88.9" y="144.78" size="1.778" layer="95" font="vector" rot="MR270"/>
 </segment>
 </net>
 <net name="MISO" class="0">
 <segment>
-<pinref part="JP1" gate="JP1" pin="MISO"/>
-<wire x1="63.5" y1="142.24" x2="73.66" y2="142.24" width="0.1524" layer="91"/>
-<label x="73.66" y="142.24" size="1.778" layer="95" font="vector" rot="MR0"/>
+<wire x1="170.18" y1="124.46" x2="160.02" y2="124.46" width="0.1524" layer="91"/>
+<label x="160.02" y="124.46" size="1.778" layer="95" font="vector"/>
+<pinref part="J2" gate="G$1" pin="7"/>
 </segment>
 <segment>
-<pinref part="M1" gate="G$1" pin="MISO"/>
-<wire x1="160.02" y1="119.38" x2="149.86" y2="119.38" width="0.1524" layer="91"/>
-<label x="149.86" y="119.38" size="1.778" layer="95" font="vector"/>
+<pinref part="J1" gate="A" pin="21"/>
+<wire x1="91.44" y1="124.46" x2="91.44" y2="111.76" width="0.1524" layer="91"/>
+<label x="91.44" y="111.76" size="1.778" layer="95" font="vector" rot="R90"/>
 </segment>
 </net>
 <net name="MOSI" class="0">
 <segment>
-<pinref part="JP1" gate="JP1" pin="MOSI"/>
-<wire x1="63.5" y1="139.7" x2="73.66" y2="139.7" width="0.1524" layer="91"/>
-<label x="73.66" y="139.7" size="1.778" layer="95" font="vector" rot="MR0"/>
+<wire x1="195.58" y1="127" x2="185.42" y2="127" width="0.1524" layer="91"/>
+<label x="195.58" y="127" size="1.778" layer="95" font="vector" rot="MR0"/>
+<pinref part="J2" gate="G$1" pin="6"/>
 </segment>
 <segment>
-<pinref part="M1" gate="G$1" pin="MOSI"/>
-<wire x1="160.02" y1="121.92" x2="149.86" y2="121.92" width="0.1524" layer="91"/>
-<label x="149.86" y="121.92" size="1.778" layer="95" font="vector"/>
+<pinref part="J1" gate="A" pin="19"/>
+<wire x1="88.9" y1="124.46" x2="88.9" y2="111.76" width="0.1524" layer="91"/>
+<label x="88.9" y="111.76" size="1.778" layer="95" font="vector" rot="R90"/>
 </segment>
 </net>
 <net name="SCK" class="0">
 <segment>
-<pinref part="JP1" gate="JP1" pin="SCLK"/>
-<wire x1="63.5" y1="144.78" x2="73.66" y2="144.78" width="0.1524" layer="91"/>
-<label x="73.66" y="144.78" size="1.778" layer="95" font="vector" rot="MR0"/>
+<wire x1="170.18" y1="127" x2="160.02" y2="127" width="0.1524" layer="91"/>
+<label x="160.02" y="127" size="1.778" layer="95" font="vector"/>
+<pinref part="J2" gate="G$1" pin="5"/>
 </segment>
 <segment>
-<pinref part="M1" gate="G$1" pin="SCK"/>
-<wire x1="160.02" y1="124.46" x2="149.86" y2="124.46" width="0.1524" layer="91"/>
-<label x="149.86" y="124.46" size="1.778" layer="95" font="vector"/>
+<pinref part="J1" gate="A" pin="23"/>
+<wire x1="93.98" y1="124.46" x2="93.98" y2="111.76" width="0.1524" layer="91"/>
+<label x="93.98" y="111.76" size="1.778" layer="95" font="vector" rot="R90"/>
 </segment>
 </net>
 <net name="CSN" class="0">
 <segment>
-<pinref part="JP1" gate="JP1" pin="CE0"/>
-<wire x1="63.5" y1="137.16" x2="73.66" y2="137.16" width="0.1524" layer="91"/>
-<label x="73.66" y="137.16" size="1.778" layer="95" font="vector" rot="MR0"/>
+<wire x1="195.58" y1="129.54" x2="185.42" y2="129.54" width="0.1524" layer="91"/>
+<label x="195.58" y="129.54" size="1.778" layer="95" font="vector" rot="MR0"/>
+<pinref part="J2" gate="G$1" pin="4"/>
 </segment>
 <segment>
-<pinref part="M1" gate="G$1" pin="CSN"/>
-<wire x1="160.02" y1="127" x2="149.86" y2="127" width="0.1524" layer="91"/>
-<label x="149.86" y="127" size="1.778" layer="95" font="vector"/>
+<pinref part="J1" gate="A" pin="24"/>
+<wire x1="93.98" y1="132.08" x2="93.98" y2="144.78" width="0.1524" layer="91"/>
+<label x="93.98" y="144.78" size="1.778" layer="95" font="vector" rot="MR270"/>
 </segment>
 </net>
 <net name="CE" class="0">
 <segment>
-<pinref part="JP1" gate="JP1" pin="GP22"/>
-<wire x1="63.5" y1="121.92" x2="73.66" y2="121.92" width="0.1524" layer="91"/>
-<label x="73.66" y="121.92" size="1.778" layer="95" font="vector" rot="MR0"/>
+<wire x1="160.02" y1="129.54" x2="170.18" y2="129.54" width="0.1524" layer="91"/>
+<label x="160.02" y="129.54" size="1.778" layer="95" font="vector"/>
+<pinref part="J2" gate="G$1" pin="3"/>
 </segment>
 <segment>
-<pinref part="M1" gate="G$1" pin="CE"/>
-<wire x1="160.02" y1="129.54" x2="149.86" y2="129.54" width="0.1524" layer="91"/>
-<label x="149.86" y="129.54" size="1.778" layer="95" font="vector"/>
+<pinref part="J1" gate="A" pin="15"/>
+<wire x1="83.82" y1="124.46" x2="83.82" y2="111.76" width="0.1524" layer="91"/>
+<label x="83.82" y="111.76" size="1.778" layer="95" font="vector" rot="R90"/>
 </segment>
 </net>
